File: 6S5P_BMS/6S5P_BMS/_autosave-6S5P_BMS.kicad_sch (KiCad schematic)
At the start: 38 parts, among them J1 Screw_Terminal_01x06, J2 Screw_Terminal_01x02, Q1 AO3414, Q2 AO3414, Q3 AO3414, Q4 AO3414, Q5 AO3414, Q6 AO3414, U1 PBQ41Z90PVPT

Commit message: Added current sensing and temperature sensing components
300u ohm shunt resistor
10k ohm thermistor at 25°C
Connections:
- net VC16 is gone; now on net Vin: C_bal1.1, R_top1.2, U1.64 (VC16)
- net Vcc: no longer U1.59 (VCC)
- net Vin: now reaches U1.63 (BAT)
